Commit message: visualize imu and camera, simplize xacro code.

File: simulation/model/turtlebot3_waffle_pi.gazebo.xacro (robot description, xacro)
@@ -1,6 +1,4 @@
 <?xml version="1.0"?>
 <robot name="turtlebot3_waffle_pi_sim" xmlns:xacro="http://ros.org/wiki/xacro">
-  <xacro:arg name="camera_visual" default="false"/>
-  <xacro:arg name="imu_visual"    default="false"/>
   <gazebo reference="base_link">
     <material>Gazebo/DarkGrey</material>
@@ -44,11 +42,4 @@
     <material>Gazebo/FlatBlack</material>
   </gazebo>
-  <gazebo reference="imu_link">
-    <sensor type="imu" name="imu">
-      <always_on>true</always_on>
-      <visualize>$(arg imu_visual)</visualize>
-    </sensor>
-    <material>Gazebo/Grey</material>
-  </gazebo>
   <gazebo>
     <plugin name="turtlebot3_waffle_pi_controller" filename="libgazebo_ros_diff_drive.so">
@@ -72,4 +63,11 @@
       <rosDebugLevel>na</rosDebugLevel>
     </plugin>
+  </gazebo>
+  <gazebo reference="imu_link">
+    <sensor type="imu" name="imu">
+      <always_on>true</always_on>
+      <visualize>true</visualize>
+    </sensor>
+    <material>Gazebo/SkyBlue</material>
   </gazebo>
   <gazebo>
@@ -101,13 +99,13 @@
     </plugin>
   </gazebo>
-<!--link : https://www.raspberrypi.org/documentation/hardware/camera/-->
-  <gazebo reference="camera_rgb_frame">
+  <!--link : https://www.raspberrypi.org/documentation/hardware/camera/-->
+  <gazebo reference="camera_link">
+    <material>Gazebo/Yellow</material>
     <sensor type="camera" name="camera1">
-      <!-- <update_rate>30.0</update_rate> -->
       <camera name='__default__'>
         <horizontal_fov>1.8</horizontal_fov>
         <image>
           <width>640</width>
-           <height>480</height>
+          <height>480</height>
           <!-- <format>R8G8B8</format> -->
         </image>
@@ -123,25 +121,13 @@
       </camera>
       <update_rate>60</update_rate>
-        <alwaysOn>1</alwaysOn>
-         <visualize>0</visualize>
+      <alwaysOn>true</alwaysOn>
+      <visualize>true</visualize>
       <plugin name="camera_controller" filename="/usr/local/lib/libgazebo_dvs_plugin.so">
-        <!-- <alwaysOn>true</alwaysOn> -->
-        <!-- <alwaysOn>1</alwaysOn> -->
-        <!-- <update_rate>60</update_rate> -->
-         <!-- <visualize>0</visualize> -->
-        <!-- <updateRate>0.0</updateRate> -->
         <eventThreshold>10</eventThreshold>
         <cameraName>camera1</cameraName>
         <robotNamespace>/</robotNamespace>
-        <!-- <imageTopicName>image_raw</imageTopicName> -->
         <eventsTopicName>events</eventsTopicName>
         <cameraInfoTopicName>camera_info</cameraInfoTopicName>
         <!-- <frameName>camera_rgb_optical_frame</frameName> -->
-        <!-- <hackBaseline>0.07</hackBaseline> -->
-        <!-- <distortionK1>0.0</distortionK1> -->
-        <!-- <distortionK2>0.0</distortionK2> -->
-        <!-- <distortionK3>0.0</distortionK3> -->
-        <!-- <distortionT1>0.0</distortionT1> -->
-        <!-- <distortionT2>0.0</distortionT2> -->
       </plugin>
       <plugin name="camera_controller" filename="libgazebo_ros_camera.so">

File: simulation/model/turtlebot3_waffle_pi.urdf.xacro (robot description, xacro)
@@ -4,4 +4,6 @@
   <xacro:include filename="$(find simulation)/model/turtlebot3_waffle_pi.gazebo.xacro"/>
   <xacro:property name="gpu" value="$(arg gpu)" />
+  <xacro:property name="imu_radius" value="0.03"/>
+	<xacro:property name="imu_length" value="0.02"/>
   <link name="base_footprint"/>
   <joint name="base_joint" type="fixed">
@@ -131,31 +133,60 @@
     <parent link="base_link"/>
     <child link="imu_link"/>
-    <origin xyz="0.0 0 0.068" rpy="0 0 0"/>
+    <origin xyz="0.0 0 0.102" rpy="0 0 0"/>
   </joint>
-  <link name="imu_link"/>
+  <link name="imu_link">
+    <!-- <inertial>
+      <mass value="0.1" />
+      <origin xyz="0 0 0" />
+      <inertia ixx="0.01" ixy="0.0" ixz="0.0"
+						 iyy="0.01" iyz="0.0"
+             izz="0.01" />
+    </inertial> -->
+    <visual>
+      <origin xyz=" 0 0 0 " rpy="0 0 0" />
+			<geometry>
+				<cylinder length="${imu_length}" radius="${imu_radius}"/>
+			</geometry>
+			<material name="green"/>
+		</visual>
+    <collision>
+			<origin xyz="0.0 0.0 0.0" rpy="0 0 0" />
+			<geometry>
+				<cylinder length="${imu_length}" radius="${imu_radius}"/>
+			</geometry>
+		</collision>
+  </link>
   <joint name="camera_joint" type="fixed">
-    <origin xyz="0.073 -0.011 0.084" rpy="0 0 0"/>
+    <origin xyz="0.07 0 0.102" rpy="0 0 0"/>
     <parent link="base_link"/>
     <child link="camera_link"/>
   </joint>
   <link name="camera_link">
+    <!-- <inertial>
+      <mass value="0.1" />
+      <origin xyz="0 0 0" />
+      <inertia ixx="0.01" ixy="0.0" ixz="0.0"
+						 iyy="0.01" iyz="0.0"
+             izz="0.01" />
+    </inertial> -->
+    <visual>
+      <origin xyz=" 0 0 0 " rpy="0 0 0" />
+			<geometry>
+				<box size="0.01 0.04 0.02"/>
+			</geometry>
+			<material name="black"/>
+		</visual>
     <collision>
-      <origin xyz="0.005 0.011 0.013" rpy="0 0 0"/>
-      <geometry>
-        <box size="0.015 0.030 0.027"/>
-      </geometry>
-    </collision>
+			<origin xyz="0.0 0.0 0.0" rpy="0 0 0" />
+			<geometry>
+				<box size="0.01 0.04 0.02"/>
+			</geometry>
+		</collision>
   </link>
-  <joint name="camera_rgb_joint" type="fixed">
-    <origin xyz="0.003 0.011 0.009" rpy="0 0 0"/>
-    <parent link="camera_link"/>
-    <child link="camera_rgb_frame"/>
-  </joint>
-  <link name="camera_rgb_frame"/>
-  <joint name="camera_rgb_optical_joint" type="fixed">
+  <!-- <joint name="camera_rgb_optical_joint" type="fixed">
     <origin xyz="0 0 0" rpy="-1.57 0 -1.57"/>
     <parent link="camera_rgb_frame"/>
     <child link="camera_rgb_optical_frame"/>
   </joint>
-  <link name="camera_rgb_optical_frame"/>
+  <link name="camera_rgb_optical_frame"/> -->
 </robot>
