Commit message: 2022-04-25

File: simulation/model/turtlebot3_waffle_pi.urdf.xacro (robot description, xacro)
@@ -184,9 +184,3 @@
 		</collision>
   </link>
-  <!-- <joint name="camera_rgb_optical_joint" type="fixed">
-    <origin xyz="0 0 0" rpy="-1.57 0 -1.57"/>
-    <parent link="camera_rgb_frame"/>
-    <child link="camera_rgb_optical_frame"/>
-  </joint>
-  <link name="camera_rgb_optical_frame"/> -->
 </robot>
